File: lueftermonster.kicad_sch (KiCad schematic)
At the start: 87 parts, among them J1 Barrel_Jack, J10 Fan, J11 Fan, J12 Fan, J13 Fan, J14 Fan, J15 Fan, J16 Fan, J17 PROG, J2 Fan, J3 Fan, J4 Fan, J5 Fan, J6 Fan, J7 Fan, J8 Fan, J9 Fan, Q1 Q_PMOS_GSD, Q2 Q_NMOS_GSD, Q3 Q_NMOS_GSD, Q4 Q_NMOS_GSD, Q5 Q_NMOS_GSD, U1 ESP32-WROOM-32E, U2 AOZ1280CI, U3 AMS1117-5.0

Commit message: more bom
Parts:
- C1, C3: value TBD -> 100n; footprint Capacitor_SMD:C_0402_1005Metric -> Capacitor_SMD:C_0805_2012Metric; LCSC (none) -> C28233; now fitted
- C10, C2, C26, C8: LCSC (none) -> C440198; MPN C0805C106K4PACTU -> GRM21BR61H106KE43L; Manufacturer KEMET -> Murata Electronics
- C6, C7: footprint Capacitor_SMD:C_0805_2012Metric -> Capacitor_SMD:C_1206_3216Metric; LCSC (none) -> C29823; MPN (none) -> 1206B475K500NT; Manufacturer (none) -> FH (Guangdong Fenghua Advanced Tech)
- D2: Digikey 1655-1928-1-ND -> (none); LCSC (none) -> C8598; MPN DSS15UTR -> B5819W SL; Manufacturer SMC Diode Solutions -> Jiangsu Changjing Electronics Technology Co., Ltd.
- FB1, FB2: value 30R @ 100MHz -> 120R @ 100MHz; footprint Inductor_SMD:L_0603_1608Metric -> Inductor_SMD:L_1206_3216Metric; Digikey 490-5447-1-ND -> (none); LCSC (none) -> C337884; MPN BLM18KG300TN1D -> BLM31KN121SN1L
- R1, R16, R17, R18, R19, R2, R20, R21, R22, R23, R24, R25, R26, R27, R28, R29, R30, R5: LCSC (none) -> C25744; MPN (none) -> 0402WGF1002TCE; Manufacturer (none) -> UNI-ROYAL(Uniroyal Elec)
- R10, R11: LCSC (none) -> C21189; MPN (none) -> 0603WAF0000T5E; Manufacturer (none) -> UNI-ROYAL(Uniroyal Elec)
- R12, R13, R14, R15: LCSC (none) -> C11702; MPN (none) -> 0402WGF1001TCE; Manufacturer (none) -> UNI-ROYAL(Uniroyal Elec)
Connections:
- net +12V: now also FB1.2; no longer FB1.1
- net at C1.1, Q1.1 (S), Q1.2 (S)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: now also FB1.1; no longer FB1.2
Other:
- moved on the sheet: D1, F1, J1, Q1, R1
