File: lueftermonster.kicad_sch (KiCad schematic)
At the start: 96 parts, among them J1 Barrel_Jack, J10 Fan, J11 Fan, J12 Fan, J13 Fan, J14 Fan, J15 Fan, J16 Fan, J17 PROG, J18 W1, J19 W1, J2 Fan, J20 W1, J21 W1, J3 Fan, J4 Fan, J5 Fan, J6 Fan, J7 Fan, J8 Fan, J9 Fan, Q1 Q_PMOS_GSD, Q2 Q_NMOS_GSD, Q3 Q_NMOS_GSD, Q4 Q_NMOS_GSD, U1 ESP32-WROOM-32E, U2 AOZ1280CI, U3 AMS1117-5.0

Commit message: snap
Parts:
- gave numbers to parts that had none: 2
Connections:
- net PWM: now also U1.37 (IO23); no longer U1.16 (IO13)
- net TACH1: now also U1.36 (IO22); no longer U1.37 (IO23)
- net TACH11: now also U1.13 (IO14); no longer U1.9 (IO33)
- net TACH12: now also U1.12 (IO27); no longer U1.10 (IO25)
- net TACH14: now also U1.10 (IO25); no longer U1.12 (IO27)
- net TACH15: now also U1.9 (IO33); no longer U1.13 (IO14)
- net TACH2: now also U1.33 (IO21); no longer U1.36 (IO22)
- net TACH3: now also U1.31 (IO19); no longer U1.33 (IO21)
- net TACH4: now also U1.30 (IO18); no longer U1.31 (IO19)
- net TACH5: now also U1.28 (IO17); no longer U1.30 (IO18)
- net TACH6: now also U1.27 (IO16); no longer U1.28 (IO17)
- net TACH7: now also U1.26 (IO4); no longer U1.27 (IO16)
- net W1: now also U1.16 (IO13); no longer U1.26 (IO4)
Changed lines of the file:
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@@
 	)
 	(label "TACH1"
-		(at 62.23 123.19 0)
+		(at 62.23 120.65 0)
 		(fields_autoplaced yes)
 		(effects
@@
 	)
 	(label "TACH5"
-		(at 62.23 113.03 0)
+		(at 62.23 110.49 0)
 		(fields_autoplaced yes)
 		(effects
@@
 	)
 	(label "TACH3"
-		(at 62.23 118.11 0)
+		(at 62.23 115.57 0)
 		(fields_autoplaced yes)
 		(effects
@@
 	)
 	(label "TACH15"
-		(at 62.23 102.87 0)
+		(at 62.23 135.89 0)
 		(fields_autoplaced yes)
 		(effects
@@
 	)
 	(label "TACH7"
-		(at 62.23 107.95 0)
+		(at 62.23 92.71 0)
 		(fields_autoplaced yes)
 		(effects
@@
 	)
 	(label "TACH14"
-		(at 62.23 130.81 0)
+		(at 62.23 125.73 0)
 		(fields_autoplaced yes)
 		(effects
@@
 	)
 	(label "TACH6"
-		(at 62.23 110.49 0)
+		(at 62.23 107.95 0)
 		(fields_autoplaced yes)
 		(effects
@@
 	)
 	(label "TACH4"
-		(at 62.23 115.57 0)
+		(at 62.23 113.03 0)
 		(fields_autoplaced yes)
 		(effects
@@
 	)
 	(label "W1"
-		(at 62.23 92.71 0)
+		(at 62.23 100.33 0)
 		(fields_autoplaced yes)
 		(effects
@@
 	)
 	(label "PWM"
-		(at 62.23 100.33 0)
+		(at 62.23 123.19 0)
 		(fields_autoplaced yes)
 		(effects
@@
 	)
 	(label "TACH2"
-		(at 62.23 120.65 0)
+		(at 62.23 118.11 0)
 		(fields_autoplaced yes)
 		(effects
@@
 	)
 	(label "TACH11"
-		(at 62.23 135.89 0)
+		(at 62.23 102.87 0)
 		(fields_autoplaced yes)
 		(effects
@@
 	)
 	(label "TACH12"
-		(at 62.23 125.73 0)
+		(at 62.23 130.81 0)
 		(fields_autoplaced yes)
 		(effects
@@
 		(dnp no)
 		(fields_autoplaced yes)
-		(property "Reference" "C?"
+		(property "Reference" "C4"
 			(at 23.0759 85.1541 0)
 			(effects
@@
 			(project "lueftermonster"
 				(path "/ae70ba22-ffaf-465a-806a-dbca86e4d278"
-					(reference "C?")
+					(reference "C4")
 					(unit 1)
 				)
@@
 		(on_board yes)
 		(dnp no)
-		(property "Reference" "R?"
+		(property "Reference" "R33"
 			(at 23.9014 76.2578 0)
 			(effects
@@
 			(project "lueftermonster"
 				(path "/ae70ba22-ffaf-465a-806a-dbca86e4d278"
-					(reference "R?")
+					(reference "R33")
 					(unit 1)
 				)

Commit message: update bom
Parts:
- J18, J19, J20, J21: LCSC (none) -> C2883760; MPN (none) -> X6511WVS-03H-C60D48R2; Manufacturer (none) -> XKB Connection
- R9: value TBD -> 4k7; LCSC (none) -> C25900; MPN (none) -> 0402WGF4701TCE; Manufacturer (none) -> UNI-ROYAL(Uniroyal Elec)
Changed lines of the file:
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@@
 			)
 		)
+		(property "LCSC" "C2883760"
+			(at 72.39 170.18 0)
+			(effects
+				(font
+					(size 1.27 1.27)
+				)
+				(hide yes)
+			)
+		)
+		(property "MPN" "X6511WVS-03H-C60D48R2"
+			(at 72.39 170.18 0)
+			(effects
+				(font
+					(size 1.27 1.27)
+				)
+				(hide yes)
+			)
+		)
+		(property "Manufacturer" "XKB Connection"
+			(at 72.39 170.18 0)
+			(effects
+				(font
+					(size 1.27 1.27)
+				)
+				(hide yes)
+			)
+		)
 		(pin "1"
 		)
@@
 			)
 		)
+		(property "LCSC" "C2883760"
+			(at 93.98 170.18 0)
+			(effects
+				(font
+					(size 1.27 1.27)
+				)
+				(hide yes)
+			)
+		)
+		(property "MPN" "X6511WVS-03H-C60D48R2"
+			(at 93.98 170.18 0)
+			(effects
+				(font
+					(size 1.27 1.27)
+				)
+				(hide yes)
+			)
+		)
+		(property "Manufacturer" "XKB Connection"
+			(at 93.98 170.18 0)
+			(effects
+				(font
+					(size 1.27 1.27)
+				)
+				(hide yes)
+			)
+		)
 		(pin "1"
 		)
@@
 			)
 		)
+		(property "LCSC" "C2883760"
+			(at 93.98 187.96 0)
+			(effects
+				(font
+					(size 1.27 1.27)
+				)
+				(hide yes)
+			)
+		)
+		(property "MPN" "X6511WVS-03H-C60D48R2"
+			(at 93.98 187.96 0)
+			(effects
+				(font
+					(size 1.27 1.27)
+				)
+				(hide yes)
+			)
+		)
+		(property "Manufacturer" "XKB Connection"
+			(at 93.98 187.96 0)
+			(effects
+				(font
+					(size 1.27 1.27)
+				)
+				(hide yes)
+			)
+		)
 		(pin "1"
 		)
@@
 			)
 		)
+		(property "LCSC" "C2883760"
+			(at 72.39 187.96 0)
+			(effects
+				(font
+					(size 1.27 1.27)
+				)
+				(hide yes)
+			)
+		)
+		(property "MPN" "X6511WVS-03H-C60D48R2"
+			(at 72.39 187.96 0)
+			(effects
+				(font
+					(size 1.27 1.27)
+				)
+				(hide yes)
+			)
+		)
+		(property "Manufacturer" "XKB Connection"
+			(at 72.39 187.96 0)
+			(effects
+				(font
+					(size 1.27 1.27)
+				)
+				(hide yes)
+			)
+		)
 		(pin "1"
 		)
@@
 			)
 		)
-		(property "Value" "TBD"
+		(property "Value" "4k7"
 			(at 128.4986 167.5821 0)
 			(effects
@@
 			(at 127 166.37 0)
 			(effects
+				(font
+					(size 1.27 1.27)
+				)
+				(hide yes)
+			)
+		)
+		(property "Manufacturer" "UNI-ROYAL(Uniroyal Elec)"
+			(at 127 166.37 0)
+			(effects
+				(font
+					(size 1.27 1.27)
+				)
+				(hide yes)
+			)
+		)
+		(property "MPN" "0402WGF4701TCE"
+			(at 127 166.37 0)
+			(effects
+				(font
+					(size 1.27 1.27)
+				)
+				(hide yes)
+			)
+		)
+		(property "Digikey" ""
+			(at 127 166.37 0)
+			(effects
+				(font
+					(size 1.27 1.27)
+				)
+				(hide yes)
+			)
+		)
+		(property "Spec" ""
+			(at 127 166.37 0)
+			(effects
+				(font
+					(size 1.27 1.27)
+				)
+				(hide yes)
+			)
+		)
+		(property "Notes" ""
+			(at 127 166.37 0)
+			(effects
+				(font
+					(size 1.27 1.27)
+				)
+				(hide yes)
+			)
+		)
+		(property "LCSC" "C25900"
+			(at 127 166.37 0)
+			(effects

Commit message: replace out of stock 1R 0402
Parts:
- R6, R7, R8: LCSC C25086 -> C102864; MPN 0402WGF100KTCE -> RTT021R00FTH; Manufacturer UNI-ROYAL(Uniroyal Elec) -> RALEC
Changed lines of the file:
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@@
 			)
 		)
-		(property "LCSC" "C25086"
+		(property "LCSC" "C102864"
 			(at 99.06 123.19 0)
 			(effects
@@
 			)
 		)
-		(property "MPN" "0402WGF100KTCE"
+		(property "MPN" "RTT021R00FTH"
 			(at 99.06 123.19 0)
 			(effects
@@
 			)
 		)
-		(property "Manufacturer" "UNI-ROYAL(Uniroyal Elec)"
+		(property "Manufacturer" "RALEC"
 			(at 99.06 123.19 0)
 			(effects
@@
 			)
 		)
-		(property "LCSC" "C25086"
+		(property "LCSC" "C102864"
 			(at 99.06 100.33 0)
 			(effects
@@
 			)
 		)
-		(property "MPN" "0402WGF100KTCE"
+		(property "MPN" "RTT021R00FTH"
 			(at 99.06 100.33 0)
 			(effects
@@
 			)
 		)
-		(property "Manufacturer" "UNI-ROYAL(Uniroyal Elec)"
+		(property "Manufacturer" "RALEC"
 			(at 99.06 100.33 0)
 			(effects
@@
 			)
 		)
-		(property "LCSC" "C25086"
+		(property "LCSC" "C102864"
 			(at 99.06 146.05 0)
 			(effects
@@
 			)
 		)
-		(property "MPN" "0402WGF100KTCE"
+		(property "MPN" "RTT021R00FTH"
 			(at 99.06 146.05 0)
 			(effects
@@
 			)
 		)
-		(property "Manufacturer" "UNI-ROYAL(Uniroyal Elec)"
+		(property "Manufacturer" "RALEC"
 			(at 99.06 146.05 0)
 			(effects
