File: lueftermonster.kicad_pcb (KiCad board)
At the start: 2 copper layers, 94 x 60 mm, 96 parts, among them J1 Barrel_Jack, J10 Fan, J11 Fan, J12 Fan, J13 Fan, J14 Fan, J15 Fan, J16 Fan, J17 PROG, J18 W1, J19 W1, J2 Fan, J20 W1, J21 W1, J3 Fan, J4 Fan, J5 Fan, J6 Fan, J7 Fan, J8 Fan, J9 Fan, Q1 Q_PMOS_GSD, Q2 Q_NMOS_GSD, Q3 Q_NMOS_GSD, Q4 Q_NMOS_GSD, U1 ESP32-WROOM-32E, U2 AOZ1280CI, U3 AMS1117-5.0

Commit message: tweaks
Routing:
- net GND: vias 187 -> 186
Other:
- board text added: "12V 2.5A max center +"
Changed lines of the file:
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@@
+		)
+	)
+	(gr_text "12V 2.5A max\ncenter +"
+		(at 104.2 100.3 0)
+		(layer "F.SilkS")
+		(effects
+			(font
+				(size 1 1)
+				(thickness 0.15)
+			)
 		)
 	)
@@
 	)
 	(via
-		(at 148.9 66.3)
-		(size 0.8)
-		(drill 0.4)
-		(layers "F.Cu" "B.Cu")
-		(free yes)
-		(net 2)
-	)
-	(via
 		(at 123.9 75.9)
 		(size 0.8)
@@
 	)
 	(via
-		(at 99.5 102)
-		(size 0.8)
-		(drill 0.4)
+		(at 98.3 101.3)
+		(size 0.8)
+		(drill 0.4)
